File: Hardware/PCB/PCB_Ted/HAL_95/HAL_95.kicad_sch (KiCad schematic)
At the start: 0 parts

Commit message: added sensors
Other:
- added sheet Motor_Driver (Motor_Driver.kicad_sch)
- added sheet Sensors (sensors.kicad_sch)
- sheet STM32 ports: added AIN1, AIN2, BIN1, BIN2, COLOR_INT, ENCA_OUT1, ENCA_OUT2, ENCB_OUT1, ENCB_OUT2, HC05_KEY, HC05_RX, HC05_STATE, HC05_TX, I2C1_SCL, I2C1_SDA, PWM_SERVO, TOF_GPIO1, TOF_XSHUT, ~{FAULT}, ~{SLEEP}; removed none
