File: Hardware/PCB/PCB_Ted/HAL_95/stm32.kicad_sch (KiCad schematic)
At the start: 23 parts, among them J1 ST_LINK, J3 NEOPIXELS, SW1 431183015816, SW2 431183015816, U1 STM32G431RBTx, Y1 16MHz

Commit message: added sensors
Parts:
- added R4: 400, Resistor_SMD:R_0402_1005Metric, symbol Device:R_Small
Connections:
- net JCLK/SWCLK: now also U1.50 (PA14); no longer U1.46 (PA12)
- net BIN1: now reaches U1.10 (PC2)
- net BIN2: now reaches U1.11 (PC3)
- net ENCB_OUT1: now reaches U1.12 (PA0)
- net ENCB_OUT2: now reaches U1.13 (PA1)
- net HC05_TX: now reaches U1.14 (PA2)
- net HC05_RX: now reaches U1.17 (PA3)
- net ENCA_OUT2: now reaches U1.18 (PA4)
- net HC05_STATE: now reaches U1.19 (PA5)
- net ENCA_OUT1: now reaches U1.20 (PA6)
- net HC05_KEY: now reaches U1.21 (PA7)
- net COLOR_INT: now reaches U1.25 (PB1)
- net at J3.2 (Pin_2): now also R4.1; no longer U1.38 (PC6)
- net ~{FAULT}: now reaches U1.41 (PC9)
- net ~{SLEEP}: now reaches U1.42 (PA8)
- net STM32_D-: now reaches U1.45 (PA11)
- net I2C1_SCL: now reaches U1.51 (PA15)
- net TOF_GPIO1: now reaches U1.55 (PD2)
- net TOF_XSHUT: now reaches U1.56 (PB3)
- net PWM_SERVO: now reaches U1.59 (PB6)
- net I2C1_SDA: now reaches U1.60 (PB7)
- net AIN1: now reaches U1.8 (PC0)
- net AIN2: now reaches U1.9 (PC1)
- new net: R4.2, U1.38 (PC6)
- new net STM32_D+: U1.46 (PA12)
Other:
- moved on the sheet: J3
