File: Hardware/PCB/PCB_Yahya/HAL95_power/Charger_BQ25896.kicad_sch (KiCad schematic)
At the start: 33 parts, among them J4 Conn_01x02_Pin, SW2 SW_Push, U2 XC6206P332MR, U5 BQ25896RTW

Commit message: Update: modification symbole
Parts:
- removed U5: BQ25896RTW, Package_DFN_QFN:Texas_RTW_WQFN-24-1EP_4x4mm_P0.5mm_EP2.7x2.7mm_ThermalVias, symbol power_lib:BQ25896RTW
- added U1: BQ25896RTW, Package_DFN_QFN:Texas_RTW_WQFN-24-1EP_4x4mm_P0.5mm_EP2.7x2.7mm_ThermalVias, symbol power_lib:BQ25896RTW
Connections:
- net +5V: now also U1.15 (SYS), U1.16 (SYS)
- net BAT: now also U1.13 (BAT), U1.14 (BAT)
- net GND: now also U1.17 (PGND), U1.18 (PGND), U1.2 (PSEL), U1.9 (~{CE})
- net INT_BQ: now also U1.7 (INT)
- net REGN: now also U1.22 (REGN)
- net STAT: now also U1.4 (STAT)
- net STM32_I2C_SCL_BQ: now also U1.5 (SCL)
- net STM32_I2C_SDA_BQ: now also U1.6 (SDA)
- net TS: now also U1.11 (TS)
- net VBUS: now also U1.1 (VBUS)
- net nQON: now also U1.12 (~{QON})
- net ~{PG}: now also U1.3 (~{PG})
- net at C13.1: now also U1.21 (BTST)
- net at C13.2, L2.1: now also U1.19 (SW), U1.20 (SW)
- net at R15.1: now also U1.10 (ILIM)
- net at C12.1: now also U1.23 (PMID)
- no-connect marks 1 -> 2
