File: Hardware/PCB/HAL_95/USB_C.kicad_sch (KiCad schematic)
At the start: 7 parts, among them J10 USB_C_Receptacle_USB2.0_14P, U4 USBLC6-2SC6

Commit message: finished schematic
Parts:
- removed F2: 250 mA, Fuse:Fuse_0603_1608Metric, symbol Device:Polyfuse_Small
- removed FB2: 120Ω@100MHz, Inductor_SMD:L_0603_1608Metric, symbol Device:FerriteBead
Connections:
- net VBUS: now also J10.A4 (VBUS), J10.A9 (VBUS), J10.B4 (VBUS), J10.B9 (VBUS)

Commit message: placing components
Changed lines of the file:
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@@
+		(color 0 0 0 0)
+	)
+	(junction
+		(at 140.97 107.95)
+		(diameter 0)
 		(color 0 0 0 0)
 	)
@@
 					(unit 1)
 				)
+			)
+		)
+	)
+	(symbol
+		(lib_id "power:PWR_FLAG")
+		(at 140.97 107.95 90)
+		(unit 1)
+		(body_style 1)
+		(exclude_from_sim no)
+		(in_bom yes)
+		(on_board yes)
+		(in_pos_files yes)
+		(dnp no)
+		(fields_autoplaced yes)
+		(property "Reference" "#FLG02"
+			(at 139.065 107.95 0)
+			(hide yes)
+			(show_name no)
+			(do_not_autoplace no)
+			(effects
+				(font
+					(size 1.27 1.27)
+				)
+			)
+		)
+		(property "Value" "PWR_FLAG"
+			(at 137.16 107.9499 90)
+			(show_name no)
+			(do_not_autoplace no)
+			(effects
+				(font
+					(size 1.27 1.27)
+				)
+				(justify left)
+			)
+		)
+		(property "Footprint" ""
+			(at 140.97 107.95 0)
+			(hide yes)
+			(show_name no)
+			(do_not_autoplace no)
+			(effects
+				(font
+					(size 1.27 1.27)
+				)
+			)
+		)
+		(property "Datasheet" ""
+			(at 140.97 107.95 0)
+			(hide yes)
+			(show_name no)
+			(do_not_autoplace no)
+			(effects
+				(font
+					(size 1.27 1.27)
+				)
+			)
+		)
+		(property "Description" "Special symbol for telling ERC where power comes from"
+			(at 140.97 107.95 0)
+			(hide yes)
+			(show_name no)
+			(do_not_autoplace no)
+			(effects
+				(font
+					(size 1.27 1.27)
+				)
+			)
+		)
+		(pin "1"
+		)
+		(instances
+			(project "HAL_95"
+				(path "/d28472ac-3b92-430d-9be8-f4bdbfbb9f17/cf868148-9de1-446f-aaa2-162914e71069"
+					(reference "#FLG02")
+					(unit 1)
+				)
