File: Hardware/PCB/HAL_95/Motor_Driver.kicad_sch (KiCad schematic)
At the start: 11 parts, among them J2 Conn_01x06, J4 Conn_01x06, J5 SERVO, U2 DRV8833PWPR

Commit message: finished schematic
Parts:
- added C32: 470u, Capacitor_SMD:CP_Elec_10x10.5, symbol Device:C_Small
- C14: value 0u01 -> 10n
- C16: JLCPCB Part # C13585 -> C76614
- R2, R3: footprint Resistor_SMD:R_0402_1005Metric -> Resistor_SMD:R_0805_2012Metric; JLCPCB Part # C270629 -> C171371
Connections:
- net SYS is gone; now on net +5V: C14.2, C16.1, U2.12 (VM)
- net +5V: now also C32.1
- net GND: now also C32.2

Commit message: reviewed schematicand ioc file
Parts:
- removed C32: 470u, Capacitor_SMD:CP_Elec_10x10.5, symbol Device:C_Small
- added C37: 470u, Capacitor_SMD:CP_Elec_10x10.5, symbol Device:C_Polarized
- added C38: 10u, Capacitor_SMD:C_0603_1608Metric, symbol Device:C_Small
- added R25: 10k, Resistor_SMD:R_0402_1005Metric, symbol Device:R_Small
- C16: footprint Capacitor_SMD:C_0402_1005Metric -> Capacitor_SMD:C_0603_1608Metric
Connections:
- net +3.3V: now also J2.2 (Pin_2), J4.2 (Pin_2), R25.1; no longer J2.5 (Pin_5), J4.5 (Pin_5)
- net +5V: now also J5.2 (Pin_2), C37.1, C38.1; no longer J5.3 (Pin_3)
- net GND: now also J2.5 (Pin_5), J4.5 (Pin_5), C37.2, C38.2; no longer J2.2 (Pin_2), J4.2 (Pin_2)
- net PWM_SERVO: now also J5.3 (Pin_3); no longer J5.2 (Pin_2)
- net ~{FAULT}: now also R25.2
Other:
- note added: "170mA, 200m, 6mW"
- note added: "A changer comme moteur du dessus !"
- moved on the sheet: C17, C18

Commit message: changed ioc and placement
Other:
- note removed: "A changer comme moteur du dessus !"
Changed lines of the file:
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@@
-		)
-	)
-	(text "A changer comme moteur du dessus !"
-		(exclude_from_sim no)
-		(at 202.184 147.828 0)
-		(effects
-			(font
-				(size 1.27 1.27)
-			)
 		)
 	)

Commit message: updated routing
Connections:
- net BOUT1: now also J4.6 (Pin_6); no longer J4.1 (Pin_1)
- net BOUT2: now also J4.1 (Pin_1); no longer J4.6 (Pin_6)
Changed lines of the file:
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@@
 	(global_label "BOUT1"
 		(shape input)
-		(at 198.12 97.79 180)
+		(at 195.58 134.62 180)
 		(fields_autoplaced yes)
 		(effects
@@
 		)
 		(property "Intersheetrefs" "${INTERSHEET_REFS}"
-			(at 189.0267 97.79 0)
+			(at 186.4867 134.62 0)
 			(hide yes)
 			(show_name no)
@@
 	(global_label "BOUT2"
 		(shape input)
-		(at 195.58 134.62 180)
+		(at 198.12 97.79 180)
 		(fields_autoplaced yes)
 		(effects
@@
 		)
 		(property "Intersheetrefs" "${INTERSHEET_REFS}"
-			(at 186.4867 134.62 0)
+			(at 189.0267 97.79 0)
 			(hide yes)
 			(show_name no)
