File: Hardware/PCB/HAL_95/HAL_95.kicad_pcb (KiCad board)
At the start: 4 copper layers, 70 x 70 mm, 106 parts, among them J1 ST_LINK, J10 USB_C_Receptacle_USB2.0_14P, J11 Conn_01x03, J12 VL53L0CXV0DH1, J2 Conn_01x06, J3 NEOPIXELS, J4 Conn_01x06, J5 SERVO, J6 ADA3595, J7 VL53L0CXV0DH1, J8 HC-05, J9 Battery, Q1 DMN313DLT-7, Q2 DMP1045U-7, Q3 MMDT2907A-7-F, SW1 USER_BTN, SW2 NRST, SW3 nQON, U1 STM32G431RBTx, U2 DRV8833PWPR, U3 BU33SD5WG-TR, U4 USBLC6-2SC6, U5 BQ25896RTW, U6 SN74AHCT1G125DBVR, U8 BQ27220YZFR, Y1 16MHz

Commit message: placing components
Parts:
- removed TP1: TestPoint, TestPoint:TestPoint_Pad_D2.0mm
- U5: footprint Package_DFN_QFN:Texas_RTW_WQFN-24-1EP_4x4mm_P0.5mm_EP2.7x2.7mm_ThermalVias -> Package_DFN_QFN:Texas_RTW_WQFN-24-1EP_4x4mm_P0.5mm_EP2.7x2.7mm
- moved J5 64.7 mm to (156.8, 62.5), turned to -90 degrees
- moved SW1 64.1 mm to (220.9, 50.8), turned to -90 degrees
- moved J3 55.8 mm to (183.7, 28.1), turned to 180 degrees
- moved C38 55.8 mm to (161.1, 61.1), turned to 90 degrees
- moved C30 49.0 mm to (182.9, 31.8), turned to 180 degrees
- moved R4 47.6 mm to (183.9, 34.0), turned to -90 degrees
- moved J12 44.9 mm to (166.1, 37.4), turned to -135 degrees
- moved J7 44.9 mm to (211.0, 37.4), turned to 135 degrees
- moved U6 42.2 mm to (183.2, 37.7), turned to 90 degrees
- moved C31 42.1 mm to (180.6, 37.7), turned to -90 degrees
- moved C13 41.1 mm to (220.9, 47.4), turned to 180 degrees
- moved C40 39.5 mm to (167.1, 42.0), turned to 45 degrees
- moved C39 39.4 mm to (206.3, 38.3), turned to -45 degrees
- moved TP4 38.0 mm to (202.7, 69.5)
- moved C10 19.9 mm to (156.7, 54.3), turned to 0 degrees
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Connections:
- C13 pad 2: Net-(U1-PC13) -> Net-(U1-PA10)
- C19 pad 1: VBUS -> +5V
- JP2 pad 2: VBUS -> +5V
- Q2 pad 3: +5V -> VBUS
- Q3 pad 4: +5V -> VBUS
- R21 pad 1: +5V -> VBUS
- SW1 pad 2: Net-(U1-PC13) -> Net-(U1-PA10)
- U1 pad 2: Net-(U1-PC13) -> unconnected-(U1-PC13-Pad2)
- U1 pad 37: /STM32/NEOPIXEL_PWM -> /STM32/BUZZER
- U1 pad 44: unconnected-(U1-PA10-Pad44) -> Net-(U1-PA10)
- U1 pad 59: /STM32/BUZZER -> /STM32/NEOPIXEL_PWM
- U5 pad 1: VBUS -> +5V
Routing:
- net +3.3V: track 0.00 -> 95.8 mm, vias 0 -> 33
- net +5V: track 0.00 -> 88.1 mm, vias 0 -> 22
- net /STM32/I2C1_SDA_TOF_COLOR: track 0.00 -> 73.0 mm, vias 0 -> 9
- net /STM32/I2C1_SCL_TOF_COLOR: track 0.00 -> 71.8 mm, vias 0 -> 4
- net VBUS: track 0.18 -> 55.0 mm, vias 1 -> 2
- net /STM32/~{RST}: track 0.00 -> 54.7 mm, vias 0 -> 4
- net /Charger_BQ25896/I2C3_SDA_FG_BQ: track 0.00 -> 49.4 mm, vias 0 -> 3
- net /STM32/BUZZER: track 0.00 -> 43.7 mm, vias 0 -> 2
- net GND: track 2.72 -> 41.9 mm, vias 0 -> 74
- net /Motor_Driver/PWM_SERVO: track 0.49 -> 37.2 mm, vias 1 -> 2
- net /Charger_BQ25896/I2C3_SCL_FG_BQ: track 0.00 -> 35.7 mm, vias 0 -> 2
- net Net-(U1-PA10): track 0.00 -> 33.7 mm, vias 0 -> 2
- net /STM32/TOF_2_XSHUT: track 0.00 -> 31.6 mm, vias 0 -> 2
- net /STM32/TOF_2_GPIO1: track 0.00 -> 31.5 mm, vias 0 -> 2
- net /Motor_Driver/ENCA_OUT1: track 0.00 -> 31.3 mm, vias 0 -> 2
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- added copper zone on In2.Cu, net +3.3V
- added copper zone on B.Cu, net +5V
- added copper zone on F.Cu, net +5V
- added copper zone on In2.Cu, net +5V
- added copper zone on F.Cu, net /Charger_BQ25896/BAT
- added copper zone on F.Cu, net CELL
- added copper zone on B.Cu, net GND
- added copper zone on F.Cu, net GND
- added copper zone on In1.Cu, net GND
- added copper zone on F.Cu, net Net-(JP1-A)
- added copper zone on B.Cu, net Net-(U2-AISEN)
- added copper zone on F.Cu, net Net-(U2-AISEN)
- added copper zone on B.Cu, net Net-(U2-BISEN)
- added copper zone on F.Cu, net Net-(U2-BISEN)

Commit message: enhanced routing
Parts:
- moved R19 0.58 mm to (199.4, 79.4)
- moved R15 0.32 mm to (200.4, 78.8)
Connections:
- U5 pad 25: (no net) -> GND
Routing:
- net VBUS: track 55.0 -> 30.4 mm, vias 2 -> 6
- net GND: track 41.9 -> 18.3 mm, vias 74 -> 164
- net +5V: track 88.1 -> 67.1 mm, vias 22 -> 20
- net Net-(C21-Pad2): track 6.92 -> 0.00 mm
- net CELL: track 7.75 -> 10.9 mm, vias 0 -> 2
- net /Charger_BQ25896/TS: track 9.96 -> 11.2 mm
- net +3.3V: track 95.8 -> 94.8 mm, vias 33 -> 30
- net /Motor_Driver/ENCB_OUT2: track 26.9 -> 27.7 mm
- net /Motor_Driver/BIN2: track 16.8 -> 17.6 mm
- net /Motor_Driver/ENCA_OUT2: track 30.2 -> 30.9 mm
- added copper zone on F.Cu, net Net-(C21-Pad2)
- added copper zone on F.Cu, net Net-(Q1-G)
- added copper zone on F.Cu, net Net-(Q3A-B1)
- added copper zone on In2.Cu, net VBUS

Commit message: updated routing
Parts:
- moved C18 3.97 mm to (172.4, 83.3), turned to 135 degrees
- moved C17 2.51 mm to (162.4, 71.3), turned to 45 degrees
Connections:
- J4 pad 1: BOUT1 -> BOUT2
- J4 pad 6: BOUT2 -> BOUT1
Routing:
- net GND: track 18.3 -> 71.3 mm, vias 164 -> 199
- net BOUT2: track 19.2 -> 0.00 mm
- net AOUT1: track 14.5 -> 0.00 mm
- net AOUT2: track 9.62 -> 0.00 mm
- net BOUT1: track 7.61 -> 0.85 mm
- net +3.3V: track 94.8 -> 88.3 mm
- net /Motor_Driver/ENCB_OUT2: track 27.7 -> 30.5 mm
- net /Motor_Driver/ENCB_OUT1: vias 0 -> 2
- net /STM32/I2C1_SDA_TOF_COLOR: vias 9 -> 7
- added copper zone on F.Cu, net AOUT1
- added copper zone on F.Cu, net AOUT2
- added copper zone on F.Cu, net BOUT1
- added copper zone on F.Cu, net BOUT2

Commit message: finished routing
Routing:
- net GND: track 71.3 -> 89.1 mm, vias 199 -> 227

Commit message: added logo
Parts:
- added G***: LOGO, LOGO, F.Cu at (170.1, 57.1)
- added G***: LOGO, LOGO, F.Cu at (170.7, 60.7)
- added H1: MountingHole_Pad, MountingHole:MountingHole_3.2mm_M3_Pad_Via, F.Cu at (163.8, 49.8)
Routing:
- net GND: track 89.1 -> 97.7 mm, vias 227 -> 234
- net /Charger_BQ25896/nQON: track 24.7 -> 25.4 mm
Other:
- board text added: "BLUETOOTH"
- board text added: "BUZZER"
- board text added: "CELL"
- board text added: "COLOR"
- board text added: "HAL 95 tedx"
- board text added: "MOTOR 1"
- board text added: "MOTOR 2"
- board text added: "NEOXIPEL"
- board text added: "NRST"
- board text added: "SERVO"
- board text added: "SHTDN"
- board text added: "TOF 1"
- board text added: "TOF 2"
- board text added: "USER_BTN"

Commit message: routing done
Parts:
- moved G*** 50.3 mm to (219.3, 67.4)
- moved G*** 50.3 mm to (219.9, 70.9)
Connections:
- U1 pad 26: /Charger_BQ25896/nQON -> unconnected-(U1-PB2-Pad26)
- U1 pad 36: unconnected-(U1-PB14-Pad36) -> /Charger_BQ25896/nQON
Routing:
- net SYS: track 19.3 -> 0.53 mm
- net Net-(JP1-A): track 17.7 -> 0.00 mm
- net /Charger_BQ25896/nQON: track 25.4 -> 31.9 mm
- net +3.3V: track 88.3 -> 82.4 mm, vias 30 -> 32
- net CELL: track 10.9 -> 7.81 mm, vias 2 -> 3
- net VBUS: track 30.4 -> 31.2 mm
- net /STM32/TOF_2_GPIO1: track 31.5 -> 32.1 mm
- net GND: track 97.7 -> 97.8 mm, vias 234 -> 273
- added copper zone on F.Cu, net +3.3V
- added copper zone on B.Cu, net CELL
- added copper zone on F.Cu, net SYS
