File: Hardware/PCB/HAL_95/HAL_95.kicad_pcb (KiCad board)
At the start: 4 copper layers, 70 x 70 mm, 109 parts, among them J1 ST_LINK, J10 USB_C_Receptacle_USB2.0_14P, J11 Conn_01x03, J12 VL53L0CXV0DH1, J2 Conn_01x06, J3 NEOPIXELS, J4 Conn_01x06, J5 SERVO, J6 ADA3595, J7 VL53L0CXV0DH1, J8 HC-05, J9 Battery, Q1 DMN313DLT-7, Q2 DMP1045U-7, Q3 MMDT2907A-7-F, SW1 USER_BTN, SW2 NRST, SW3 nQON, U1 STM32G431RBTx, U2 DRV8833PWPR, U3 BU33SD5WG-TR, U4 USBLC6-2SC6, U5 BQ25896RTW, U6 SN74AHCT1G125DBVR, U8 BQ27220YZFR, Y1 16MHz

Commit message: fixed routing
Routing:
- net Net-(J3-Pin_2): track 6.58 -> 8.25 mm
- net /Charger_BQ25896/nQON: track 32.6 -> 34.1 mm
- net /Charger_BQ25896/I2C3_SDA_FG_BQ: track 49.4 -> 47.9 mm
- net GND: track 98.0 -> 96.6 mm, vias 527 -> 524
- net /STM32/I2C1_SDA_TOF_COLOR: track 73.0 -> 73.9 mm
