File: Hardware/PCB/HAL_95/stm32.kicad_sch (KiCad schematic)
At the start: 24 parts, among them J1 ST_LINK, J3 NEOPIXELS, SW1 431183015816, SW2 431183015816, U1 STM32G431RBTx, Y1 16MHz

Commit message: finished schematic
Parts:
- removed JP1, JP2: SolderJumper_2_Open, Jumper:SolderJumper-2_P1.3mm_Open_TrianglePad1.0x1.5mm, symbol Jumper:SolderJumper_2_Open
- removed SW1, SW2: 431183015816, Switch_SMD_Wurth:SW_Wurth_WS-TASV_431183015816, symbol Switch_Wurth_WS-TASV:431183015816
- added C30: 470u, Capacitor_SMD:CP_Elec_10x10.5, symbol Device:C_Small
- added C31: 100n, Capacitor_SMD:C_0402_1005Metric, symbol Device:C_Small
- added SW1: USER_BTN, Button_Switch_SMD:SW_Push_1P1T_NO_CK_KMR2, symbol Switch:SW_Push
- added SW2: NRST, Button_Switch_SMD:SW_Push_1P1T_NO_CK_KMR2, symbol Switch:SW_Push
- added U6: SN74AHCT1G125DBVR, Package_TO_SOT_SMD:SOT-23-5, symbol 74xGxx:74AHCT1G125
Connections:
- net +5V: now also C30.1, C31.1, U6.5 (VCC)
- net GND: now also C10.1, C13.1, C30.2, C31.2, SW1.1, SW2.1, U6.1, U6.3 (GND)
- net VCP_RX: now also J1.13 (VCP_RX)
- net VCP_TX: now also J1.14 (VCP_TX)
- net ~{RST}: now also SW2.2
- net at C13.2, U1.53 (PC11): now also SW1.2
- net at R4.2: now also U6.4; no longer U1.38 (PC6)
- net FG_GPOUT: now reaches U1.2 (PC13)
- net I2C3_SCL_FG_BQ: now reaches U1.40 (PC8)
- net TOF_1_XSHUT: now reaches U1.54 (PC12)
- net TOF_2_GPIO1: now reaches U1.57 (PB4)
- net I2C3_SDA_FG_BQ: now reaches U1.58 (PB5)
- net BUZZER: now reaches U1.61 (PB8)
- net I2C1_SCL renamed I2C1_SCL_TOF_COLOR
- net I2C1_SDA renamed I2C1_SDA_TOF_COLOR
- net TOF_GPIO1 renamed TOF_1_GPIO1
- net TOF_XSHUT renamed TOF_2_XSHUT
- new net NEOPIXEL_PWM: U1.38 (PC6), U6.2
- no-connect marks 23 -> 15
Other:
- note added: "NEOPIXELS RING"
- moved on the sheet: C13, J1, J3, R4

Commit message: reviewed schematicand ioc file
Parts:
- C30: value 470u -> 1u; footprint Capacitor_SMD:CP_Elec_10x10.5 -> Capacitor_SMD:C_0402_1005Metric; JLCPCB Part # C96180 -> C52923
Connections:
- net +5V: now also C30.2; no longer C30.1
- net GND: now also C30.1; no longer C30.2
Other:
- moved on the sheet: C1, C2, C3, C30, C4, C5, C6, C7, C8, C9

Commit message: removed erc errors
Changed lines of the file:
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@@
 	)
 	(junction
+		(at 259.08 144.78)
+		(diameter 0)
+		(color 0 0 0 0)
+	)
+	(junction
 		(at 82.55 63.5)
 		(diameter 0)
@@
 					(unit 1)
 				)
+			)
+		)
+	)
+	(symbol
+		(lib_id "power:PWR_FLAG")
+		(at 259.08 144.78 90)
+		(unit 1)
+		(body_style 1)
+		(exclude_from_sim no)
+		(in_bom yes)
+		(on_board yes)
+		(in_pos_files yes)
+		(dnp no)
+		(fields_autoplaced yes)
+		(property "Reference" "#FLG04"
+			(at 257.175 144.78 0)
+			(hide yes)
+			(show_name no)
+			(do_not_autoplace no)
+			(effects
+				(font
+					(size 1.27 1.27)
+				)
+			)
+		)
+		(property "Value" "PWR_FLAG"
+			(at 255.27 144.7799 90)
+			(show_name no)
+			(do_not_autoplace no)
+			(effects
+				(font
+					(size 1.27 1.27)
+				)
+				(justify left)
+			)
+		)
+		(property "Footprint" ""
+			(at 259.08 144.78 0)
+			(hide yes)
+			(show_name no)
+			(do_not_autoplace no)
+			(effects
+				(font
+					(size 1.27 1.27)
+				)
+			)
+		)
+		(property "Datasheet" ""
+			(at 259.08 144.78 0)
+			(hide yes)
+			(show_name no)
+			(do_not_autoplace no)
+			(effects
+				(font
+					(size 1.27 1.27)
+				)
+			)
+		)
+		(property "Description" "Special symbol for telling ERC where power comes from"
+			(at 259.08 144.78 0)
+			(hide yes)
+			(show_name no)
+			(do_not_autoplace no)
+			(effects
+				(font
+					(size 1.27 1.27)
+				)
+			)
+		)
+		(pin "1"
+		)
+		(instances
+			(project "HAL_95"
+				(path "/d28472ac-3b92-430d-9be8-f4bdbfbb9f17/78b6ab93-d2c6-45f5-82ba-493882b68747"
+					(reference "#FLG04")
+					(unit 1)
+				)

Commit message: changed ioc and placement
Parts:
- R4: value 400 -> 300; footprint Resistor_SMD:R_0402_1005Metric -> Resistor_SMD:R_0603_1608Metric; JLCPCB Part # C11702 -> C23025
Connections:
- net BUZZER: now also U1.59 (PB6); no longer U1.61 (PB8)
- net CHARGER_INT: now also U1.33 (PB11); no longer U1.36 (PB14)
- net COLOR_INT: now also U1.58 (PB5); no longer U1.25 (PB1)
- net ENCA_OUT1: now also U1.12 (PA0); no longer U1.20 (PA6)
- net ENCA_OUT2: now also U1.13 (PA1); no longer U1.18 (PA4)
- net ENCB_OUT1: now also U1.20 (PA6); no longer U1.12 (PA0)
- net ENCB_OUT2: now also U1.18 (PA4); no longer U1.13 (PA1)
- net FG_GPOUT: now also U1.25 (PB1); no longer U1.2 (PC13)
- net HC05_RX: now also U1.23 (PC5); no longer U1.17 (PA3)
- net HC05_STATE: now also U1.24 (PB0); no longer U1.19 (PA5)
- net HC05_TX: now also U1.22 (PC4); no longer U1.14 (PA2)
- net I2C1_SCL_TOF_COLOR: now also U1.61 (PB8); no longer U1.51 (PA15)
- net I2C1_SDA_TOF_COLOR: now also U1.62 (PB9); no longer U1.60 (PB7)
- net I2C3_SDA_FG_BQ: now also U1.41 (PC9); no longer U1.58 (PB5)
- net NEOPIXEL_PWM: now also U1.37 (PB15); no longer U1.38 (PC6)
- net PWM_SERVO: now also U1.38 (PC6); no longer U1.59 (PB6)
- net VCP_RX: now also U1.53 (PC11); no longer U1.23 (PC5)
- net VCP_TX: now also U1.52 (PC10); no longer U1.22 (PC4)
- net nQON: now also U1.26 (PB2); no longer U1.34 (PB12)
- net ~{FAULT}: now also U1.17 (PA3); no longer U1.41 (PC9)
- net ~{SLEEP}: now also U1.14 (PA2); no longer U1.42 (PA8)
- net at C13.2, SW1.2: now also U1.2 (PC13); no longer U1.53 (PC11)
- net at D1.2 (A): now also U1.3 (PC14); no longer U1.33 (PB11)
Other:
- moved on the sheet: D1, R1

Commit message: placing components
Connections:
- net BUZZER: now also U1.37 (PB15); no longer U1.59 (PB6)
- net NEOPIXEL_PWM: now also U1.59 (PB6); no longer U1.37 (PB15)
- net at C13.2, SW1.2: now also U1.44 (PA10); no longer U1.2 (PC13)

Commit message: added logo
Parts:
- R4: JLCPCB Part # C23025 -> C23025
Changed lines of the file:
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@@
 			)
 		)
-		(property "JLCPCB Part #" " C23025"
+		(property "JLCPCB Part #" "C23025"
 			(at 240.03 147.32 90)
 			(hide yes)

Commit message: routing done
Connections:
- net nQON: now also U1.36 (PB14); no longer U1.26 (PB2)
Changed lines of the file:
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@@
 	)
 	(no_connect
-		(at 134.62 151.13)
+		(at 134.62 120.65)
 	)
 	(no_connect
@@
 	(wire
 		(pts
+			(xy 134.62 151.13) (xy 138.43 151.13)
+		)
+		(stroke
+			(width 0)
+			(type default)
+		)
+	)
+	(wire
+		(pts
 			(xy 138.43 128.27) (xy 134.62 128.27)
 		)
@@
 		(pts
 			(xy 233.68 85.09) (xy 233.68 86.36)
-		)
-		(stroke
-			(width 0)
-			(type default)
-		)
-	)
-	(wire
-		(pts
-			(xy 134.62 120.65) (xy 138.43 120.65)
 		)
 		(stroke
@@
 			)
 			(justify left bottom)
+		)
+	)
+	(hierarchical_label "nQON"
+		(shape input)
+		(at 138.43 151.13 0)
+		(effects
+			(font
+				(size 1.27 1.27)
+			)
+			(justify left)
 		)
 	)
@@
 		)
 	)
-	(hierarchical_label "nQON"
-		(shape input)
-		(at 138.43 120.65 0)
-		(effects
-			(font
-				(size 1.27 1.27)
-			)
-			(justify left)
-		)
-	)
