File: Hardware/PCB/HAL_95/_restore_backup_2026-10-05T12-00-09-039/Charger_BQ25896.kicad_sch (KiCad schematic)
At the start: 49 parts, among them J9 Battery, Q1 DMN313DLT-7, Q2 DMP1045U-7, Q3 MMDT2907A-7-F, SW3 nQON, U3 BU33SD5WG-TR, U5 BQ25896RTW, U8 BQ27220YZFR

Commit message: pcb done, gerber/drill files
Parts:
- TP3, TP4: now in the parts list
Changed lines of the file:
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@@
 		(in_bom yes)
 		(on_board yes)
-		(in_pos_files no)
+		(in_pos_files yes)
 		(dnp no)
 		(property "Reference" "C22"
@@
 		(body_style 1)
 		(exclude_from_sim no)
-		(in_bom no)
+		(in_bom yes)
 		(on_board yes)
 		(in_pos_files yes)
@@
 		(body_style 1)
 		(exclude_from_sim no)
-		(in_bom no)
+		(in_bom yes)
 		(on_board yes)
 		(in_pos_files yes)
