File: Hardware/PCB/HAL_95/_restore_backup_2026-10-05T12-00-09-039/Motor_Driver.kicad_sch (KiCad schematic)
At the start: 13 parts, among them J11 Conn_01x03, J12 VL53L0CXV0DH1, J6 ADA3595, J7 VL53L0CXV0DH1, J8 HC-05

Commit message: pcb done, gerber/drill files
Parts:
- removed C36, C39, C40, C41, C42: 100n, Capacitor_SMD:C_0402_1005Metric, symbol Device:C_Small
- removed H1: MountingHole_Pad, MountingHole:MountingHole_3.2mm_M3_Pad_Via, symbol Mechanical:MountingHole_Pad
- removed J11: Conn_01x03, Connector_JST:JST_GH_SM03B-GHS-TB_1x03-1MP_P1.25mm_Horizontal, symbol Connector_Generic:Conn_01x03
- removed J12, J7: VL53L0CXV0DH1, Connector_JST:JST_GH_SM06B-GHS-TB_1x06-1MP_P1.25mm_Horizontal, symbol Connector_Generic:Conn_01x06
- removed J6: ADA3595, Connector_JST:JST_GH_SM05B-GHS-TB_1x05-1MP_P1.25mm_Horizontal, symbol Connector_Generic:Conn_01x05
- removed J8: HC-05, Connector_JST:JST_GH_SM06B-GHS-TB_1x06-1MP_P1.25mm_Horizontal, symbol Connector_Generic:Conn_01x06
- removed R26, R27: 2k2, Resistor_SMD:R_0402_1005Metric, symbol Device:R
- added C14: 10n, Capacitor_SMD:C_0402_1005Metric, symbol Device:C_Small
- added C15: 2u2, Capacitor_SMD:C_0402_1005Metric, symbol Device:C_Small
- added C16, C38: 10u, Capacitor_SMD:C_0603_1608Metric, symbol Device:C_Small
- added C17, C18: 100n, Capacitor_SMD:C_0402_1005Metric, symbol Device:C_Small
- added C37: 470u, Capacitor_SMD:CP_Elec_10x10.5, symbol Device:C_Polarized
- added J2, J4: Conn_01x06, Connector_JST:JST_GH_SM06B-GHS-TB_1x06-1MP_P1.25mm_Horizontal, symbol Connector_Generic:Conn_01x06
- added J5: SERVO, Connector_JST:JST_GH_SM03B-GHS-TB_1x03-1MP_P1.25mm_Horizontal, symbol Connector_Generic:Conn_01x03
- added R2, R3: 200m, Resistor_SMD:R_0805_2012Metric, symbol Device:R_Small
- added R25: 10k, Resistor_SMD:R_0402_1005Metric, symbol Device:R_Small
- added U2: DRV8833PWPR, Package_SO:HTSSOP-16-1EP_4.4x5mm_P0.65mm_EP3.4x5mm_Mask2.46x2.31mm, symbol Driver_Motor:DRV8833PWP
Connections:
- net +3.3V: now also C17.1, C18.1, J2.2 (Pin_2), J4.2 (Pin_2), R25.1
- net +5V: now also C14.2, C16.1, C37.1, C38.1, J5.2 (Pin_2), U2.12 (VM)
- net GND: now also C15.2, C16.2, C17.2, C18.2, C37.2, C38.2, J2.5 (Pin_5), J4.5 (Pin_5), J5.1 (Pin_1), R2.2, R3.2, U2.13 (GND), U2.17 (GND)
- new net: C15.1, U2.14 (VINT)
- new net: R2.1, U2.3 (AISEN)
- new net: R3.1, U2.6 (BISEN)
- new net AIN1: U2.16 (AIN1)
- new net AIN2: U2.15 (AIN2)
- new net AOUT1: J2.1 (Pin_1), U2.2 (AOUT1)
- new net AOUT2: J2.6 (Pin_6), U2.4 (AOUT2)
- new net BIN1: U2.9 (BIN1)
- new net BIN2: U2.10 (BIN2)
- new net BOUT1: J4.6 (Pin_6), U2.7 (BOUT1)
- new net BOUT2: J4.1 (Pin_1), U2.5 (BOUT2)
- new net ENCA_OUT1: J2.3 (Pin_3)
- new net ENCA_OUT2: J2.4 (Pin_4)
- new net ENCB_OUT1: J4.3 (Pin_3)
- new net ENCB_OUT2: J4.4 (Pin_4)
- new net PWM_SERVO: J5.3 (Pin_3)
- new net VCP: C14.1, U2.11 (VCP)
- new net ~{FAULT}: R25.2, U2.8 (~{FAULT})
- new net ~{SLEEP}: U2.1 (~{SLEEP})
Other:
- note added: "170mA, 200m, 6mW"
- note added: "JST connector for Motor A"
- note added: "JST connector for Motor B"
- note added: "Motor driver"
- note added: "Servomotor"
- note removed: "BUZZER"
- note removed: "Bluetooth"
- note removed: "Color Sensor"
- note removed: "Mounting Hole"
- note removed: "TOF_1"
- note removed: "TOF_2"
- title: Sensors -> Motor Driver
