File: Hardware/PCB/HAL_95/_restore_backup_2026-10-05T12-00-09-039/USB_C.kicad_sch (KiCad schematic)
At the start: 5 parts, among them J10 USB_C_Receptacle_USB2.0_14P, U4 USBLC6-2SC6

Commit message: pcb done, gerber/drill files
Parts:
- TP2: now in the parts list
Changed lines of the file:
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@@
 		(body_style 1)
 		(exclude_from_sim no)
-		(in_bom no)
+		(in_bom yes)
 		(on_board yes)
 		(in_pos_files yes)
